File: uGSM-2G-BLE/Power.sch (KiCad schematic (older format))
At the start: 0 parts

Commit message: added tps56
Parts:
- added C? (x2): 100nF, Capacitor_SMD:C_0603_1608Metric, symbol Device:C
- added C? (x2): 10uF, Capacitor_SMD:C_1206_3216Metric, symbol Device:C
- added C? (x2): 22uF, Capacitor_SMD:C_1206_3216Metric, symbol Device:C
- added L?: 3.3uH, symbol Device:L
- added R? (x2): 10K, Resistor_SMD:R_0603_1608Metric, symbol Device:R
- added R?: 42.1K, Resistor_SMD:R_0603_1608Metric, symbol Device:R
- added U?: TPS562201DDCR, Package_TO_SOT_SMD:SOT-23-6, symbol Regulator_Switching:TPS562200
Connections:
- new net: C?.1, L?.1, U?.2 (SW)
- new net: R?.1, R?.2, U?.4 (VFB)
- new net: R?.2, U?.5 (EN)
- new net: C?.2, U?.6 (VBST)
- new net GND: C?.2, C?.2, C?.2, C?.2, C?.2, R?.1, U?.1 (GND)
- new net SIM_VCC: C?.1, C?.1, L?.2, R?.2
- new net VCC: C?.1, C?.1, C?.1, R?.1, U?.3 (VIN)
Other:
- note added: "!! check http://www.ti.com/lit/ds/symlink/tps562201.pdf Layout Guidlines !!"
- note added: "R1: 42.1k R2: 10k\nVout = 0.768 * (1+ R1/R2)\nVout = 4.00128V"
- note added: "assign footprint: L\n"
- note added: "http://www.ti.com/lit/ug/slvual5/slvual5.pdf"
