File: uGSM-2G-BLE/IO.sch (KiCad schematic (older format))
At the start: 0 parts

Commit message: removed usbl6 simcom
Parts:
- added C? (x2): 100nF, Capacitor_SMD:C_0603_1608Metric, symbol Device:C
- added D? (x2): BAT54S, Package_TO_SOT_SMD:SOT-23, symbol Diode:BAT54S
- added D?: D, symbol Device:D
- added Q?: 2N7002H, Package_TO_SOT_SMD:SOT-23, symbol Transistor_FET:2N7002H
- added R? (x3): 1k, Resistor_SMD:R_0603_1608Metric, symbol Device:R
- added R? (x5): 10k, Resistor_SMD:R_0603_1608Metric, symbol Device:R
Connections:
- net labels added: +3V3, GND, INPUT1, INPUT2
- wire segments 0 -> 26
